Commit message: camera position correction

File: franka_description/robots/hand.xacro (robot description, xacro)
@@ -87,5 +87,6 @@
       <parent link="${ns}_hand" />
       <child link="${ns}_object_link" />
-      <origin xyz="0 0 0.1034" rpy="0 0 0"/>
+      <origin xyz="0 0 0.1274" rpy="0 0 0"/>
+      <!--xyz="0 0 0.1034" rpy="0 0 0" -->
       <!-- Base delle dita 0.0584-->
    </joint>
@@ -109,5 +110,6 @@
      <!-- <origin xyz="0 0 0.0" rpy="0 ${3*pi/2} ${pi/2}"/> -->
      <!--origin xyz=" 0.04576 0.00275  0.076854" rpy="0.033641884557 -0.013806793567 1.57762792946"/-->
-     <origin xyz=" 0.04276 -0.00275  0.076854" rpy="0.033641884557 -0.013806793567 1.57762792946"/>
+     <!--origin xyz=" 0.04276 -0.00275  0.076854" rpy="0.033641884557 -0.013806793567 1.57762792946"/-->
+     <origin xyz=" 0.04276 0.002  0.065" rpy="0.033641884557 -0.013806793567 1.57762792946"/>
    </joint>
    <link name="gripper_camera">
