Commit message: update

File: franka_description/robots/end_effector/tactile_hand.xacro (robot description, xacro)
@@ -25,5 +25,5 @@
     <link name="${ns}_leftfinger">
       <visual>
-         <origin xyz="0 0 0.02" rpy="0 0 0"/>
+         <origin xyz="0 0.015 0.02" rpy="0 0 0"/>
          <geometry>
             <mesh filename="package://franka_description/meshes/tactile_finger.stl" scale="0.001 0.001 0.001"/>
@@ -42,5 +42,5 @@
     <link name="${ns}_rightfinger">
       <visual>
-         <origin xyz="0 0 0.02" rpy="0 0 ${pi}"/>
+         <origin xyz="0 -0.015 0.02" rpy="0 0 ${pi}"/>
          <geometry>
             <mesh filename="package://franka_description/meshes/tactile_finger.stl" scale="0.001 0.001 0.001"/>
@@ -75,5 +75,5 @@
       <parent link="${ns}_hand" />
       <child link="${ns}_object_link" />
-      <origin xyz="0 0 0.170" rpy="0 0 0"/>
+      <origin xyz="0 0 0.155" rpy="0 0 0"/>
       <!-- Base delle dita 0.0584-->
    </joint>
@@ -91,4 +91,23 @@
 	   </collision>
    </link>
+      <joint name="${ns}_tactile_joint" type="fixed" >
+      <parent link="${ns}_object_link" />
+      <child link="${ns}_tactile_link" />
+      <origin xyz="0 0 -0.0125" rpy="${pi/2} 0 0"/>
+      <!-- Base delle dita 0.0584-->
+   </joint>
+   <link name="${ns}_tactile_link">
+      <visual>
+         <geometry>
+            <box size="0.0 0.00 0.0"/>
+         </geometry>
+	      <material name="silver" />
+      </visual>
+      <collision>
+         <geometry>
+            <box size="0.00 0.00 0.0"/>
+         </geometry>
+	   </collision>
+   </link>
   </xacro:macro>
 </robot>

File: panda_moveit_config/config/panda_arm_tactile.srdf.xacro (robot description, xacro)
@@ -1,7 +1,3 @@
 <?xml version='1.0' encoding='utf-8'?>
-<!--This does not replace URDF, and is not an extension of URDF.
-    This is a format for representing semantic information about the robot structure.
-    A URDF file must exist for this robot as well, where the joints and the links that are referenced are defined
--->
 <robot xmlns:xacro="http://www.ros.org/wiki/xacro" name="panda">
   <xacro:include filename="$(find panda_moveit_config)/config/panda_arm.xacro" />

Commit message: pkg update

File: franka_description/robots/end_effector/tactile_hand.xacro (robot description, xacro)
@@ -75,5 +75,5 @@
       <parent link="${ns}_hand" />
       <child link="${ns}_object_link" />
-      <origin xyz="0 0 0.155" rpy="0 0 0"/>
+      <origin xyz="0 0 0.167" rpy="0 0 0"/>
       <!-- Base delle dita 0.0584-->
    </joint>
@@ -91,9 +91,10 @@
 	   </collision>
    </link>
-      <joint name="${ns}_tactile_joint" type="fixed" >
+<!-- TACTILE LINK-->
+   <joint name="${ns}_tactile_joint" type="fixed" >
       <parent link="${ns}_object_link" />
       <child link="${ns}_tactile_link" />
-      <origin xyz="0 0 -0.0125" rpy="${pi/2} 0 0"/>
-      <!-- Base delle dita 0.0584-->
+     <!-- <origin xyz="0 0 0.0" rpy="0 ${3*pi/2} ${pi/2}"/> -->
+     <origin xyz="0 0 0.0" rpy="${pi/2} 0 ${pi}"/>
    </joint>
    <link name="${ns}_tactile_link">
@@ -110,4 +111,44 @@
 	   </collision>
    </link>
+      <joint name="gripper_camera_joint" type="fixed" >
+      <parent link="${ns}_hand" />
+      <child link="gripper_camera" />
+     <!-- <origin xyz="0 0 0.0" rpy="0 ${3*pi/2} ${pi/2}"/> -->
+     <!--origin xyz=" 0.04576 0.00275  0.076854" rpy="0.033641884557 -0.013806793567 1.57762792946"/-->
+     <origin xyz=" 0.04276 -0.00275  0.076854" rpy="0.033641884557 -0.013806793567 1.57762792946"/>
+   </joint>
+   <link name="gripper_camera">
+      <visual>
+         <geometry>
+            <box size="0.0 0.00 0.0"/>
+         </geometry>
+	      <material name="silver" />
+      </visual>
+      <collision>
+         <geometry>
+            <box size="0.00 0.00 0.0"/>
+         </geometry>
+	   </collision>
+   </link>
+   <joint name="gripper_camera_visu_joint" type="fixed" >
+      <parent link="gripper_camera" />
+      <child link="gripper_camera_visu" />
+     <origin xyz=" 0.03 0.075 -0.01" rpy="-${pi/2}  0.0 ${pi} "/>
+   </joint>
+   <link name="gripper_camera_visu">
+      <visual>
+         <geometry>
+            <mesh filename="package://franka_description/meshes/Fotocamera_gripper.STL" scale="0.001 0.001 0.001"/>
+         </geometry>
+	      <material name="black">
+            <color rgba="0.5 0.5 0.5 1"/>
+         </material>
+      </visual>
+      <collision>
+         <geometry>
+            <box size="0.00 0.00 0.0"/>
+         </geometry>
+	   </collision>
+   </link>
   </xacro:macro>
 </robot>

File: panda_moveit_config/config/hand.xacro (robot description, xacro)
@@ -20,4 +20,5 @@
     <disable_collisions link1="panda_hand" link2="panda_rightfinger" reason="Adjacent" />
     <disable_collisions link1="panda_leftfinger" link2="panda_rightfinger" reason="Default" />
+    <disable_collisions link1="panda_object_link" link2="panda_tactile_link" reason="Default" />
   </xacro:macro>
 </robot>

Commit message: Addition of USB_Camera model in tactile hand

File: franka_description/robots/end_effector/tactile_hand.xacro (robot description, xacro)
@@ -131,4 +131,42 @@
 	   </collision>
    </link>
+   <joint name="realsense_camera_joint" type="fixed" >
+      <parent link="${ns}_hand" />
+      <child link="realsense_optical_frame" />
+     <origin xyz=" -0.04276 -0.00275  0.076854" rpy="0.033641884557 -0.013806793567 1.57762792946"/>
+   </joint>
+   <link name="realsense_optical_frame">
+      <visual>
+         <geometry>
+            <box size="0.0 0.00 0.0"/>
+         </geometry>
+	      <material name="silver" />
+      </visual>
+      <collision>
+         <geometry>
+            <box size="0.00 0.00 0.0"/>
+         </geometry>
+	   </collision>
+   </link>
+      <joint name="gripper_realsense_joint" type="fixed" >
+      <parent link="${ns}_hand" />
+      <child link="camera_link" />
+     <origin xyz=" -0.039278 -0.012625  0.076519" rpy= "${180*pi/180} ${-90*pi/180} 0.0" />
+     <!-- "${-1.049392*pi/180} ${-4.432421*pi/180} ${91.376356*pi/180}" -->
+     <!--"0.033641884557 -0.013806793567 1.57762792946"  -->
+   </joint>
+   <link name="camera_link">
+      <visual>
+         <geometry>
+            <box size="0.0 0.00 0.0"/>
+         </geometry>
+	      <material name="silver" />
+      </visual>
+      <collision>
+         <geometry>
+            <box size="0.00 0.00 0.0"/>
+         </geometry>
+	   </collision>
+   </link>
    <joint name="gripper_camera_visu_joint" type="fixed" >
       <parent link="gripper_camera" />

File: franka_description/robots/hand.xacro (robot description, xacro)
@@ -95,5 +95,5 @@
           <box size="0.0 0.00 0.0"/>
         </geometry>
-	<material name="silver" />
+	      <material name="silver" />
       </visual>
       <collision>
@@ -101,7 +101,85 @@
           <box size="0.00 0.00 0.0"/>
         </geometry>
-	<material name="black"/>
+	      <material name="black"/>
      </collision>
     </link>
+      <joint name="gripper_camera_joint" type="fixed" >
+      <parent link="${ns}_hand" />
+      <child link="gripper_camera" />
+     <!-- <origin xyz="0 0 0.0" rpy="0 ${3*pi/2} ${pi/2}"/> -->
+     <!--origin xyz=" 0.04576 0.00275  0.076854" rpy="0.033641884557 -0.013806793567 1.57762792946"/-->
+     <origin xyz=" 0.04276 -0.00275  0.076854" rpy="0.033641884557 -0.013806793567 1.57762792946"/>
+   </joint>
+   <link name="gripper_camera">
+      <visual>
+         <geometry>
+            <box size="0.0 0.00 0.0"/>
+         </geometry>
+	      <material name="silver" />
+      </visual>
+      <collision>
+         <geometry>
+            <box size="0.00 0.00 0.0"/>
+         </geometry>
+	   </collision>
+   </link>
+   <joint name="realsense_camera_joint" type="fixed" >
+      <parent link="${ns}_hand" />
+      <child link="realsense_optical_frame" />
+     <origin xyz=" -0.04276 -0.00275  0.076854" rpy="0.033641884557 -0.013806793567 1.57762792946"/>
+   </joint>
+   <link name="realsense_optical_frame">
+      <visual>
+         <geometry>
+            <box size="0.0 0.00 0.0"/>
+         </geometry>
+	      <material name="silver" />
+      </visual>
+      <collision>
+         <geometry>
+            <box size="0.00 0.00 0.0"/>
+         </geometry>
+	   </collision>
+   </link>
+      <joint name="gripper_realsense_joint" type="fixed" >
+      <parent link="${ns}_hand" />
+      <child link="camera_link" />
+     <origin xyz=" -0.039278 -0.012625  0.076519" rpy= "${180*pi/180} ${-90*pi/180} 0.0" />
+     <!-- "${-1.049392*pi/180} ${-4.432421*pi/180} ${91.376356*pi/180}" -->
+     <!--"0.033641884557 -0.013806793567 1.57762792946"  -->
+   </joint>
+   <link name="camera_link">
+      <visual>
+         <geometry>
+            <box size="0.0 0.00 0.0"/>
+         </geometry>
+	      <material name="silver" />
+      </visual>
+      <collision>
+         <geometry>
+            <box size="0.00 0.00 0.0"/>
+         </geometry>
+	   </collision>
+   </link>
+   <joint name="gripper_camera_visu_joint" type="fixed" >
+      <parent link="gripper_camera" />
+      <child link="gripper_camera_visu" />
+     <origin xyz=" 0.03 0.075 -0.01" rpy="-${pi/2}  0.0 ${pi} "/>
+   </joint>
+   <link name="gripper_camera_visu">
+      <visual>
+         <geometry>
+            <mesh filename="package://franka_description/meshes/Fotocamera_gripper.STL" scale="0.001 0.001 0.001"/>
+         </geometry>
+	      <material name="black">
+            <color rgba="0.5 0.5 0.5 1"/>
+         </material>
+      </visual>
+      <collision>
+         <geometry>
+            <box size="0.00 0.00 0.0"/>
+         </geometry>
+	   </collision>
+   </link>
   </xacro:macro>
 </robot>

Commit message: Remove of useless collision link

File: franka_description/robots/end_effector/tactile_hand.xacro (robot description, xacro)
@@ -105,9 +105,4 @@
 	      <material name="silver" />
       </visual>
-      <collision>
-         <geometry>
-            <box size="0.00 0.00 0.0"/>
-         </geometry>
-	   </collision>
    </link>
       <joint name="gripper_camera_joint" type="fixed" >
@@ -125,9 +120,4 @@
 	      <material name="silver" />
       </visual>
-      <collision>
-         <geometry>
-            <box size="0.00 0.00 0.0"/>
-         </geometry>
-	   </collision>
    </link>
    <joint name="realsense_camera_joint" type="fixed" >
@@ -143,9 +133,4 @@
 	      <material name="silver" />
       </visual>
-      <collision>
-         <geometry>
-            <box size="0.00 0.00 0.0"/>
-         </geometry>
-	   </collision>
    </link>
       <joint name="gripper_realsense_joint" type="fixed" >
@@ -163,9 +148,4 @@
 	      <material name="silver" />
       </visual>
-      <collision>
-         <geometry>
-            <box size="0.00 0.00 0.0"/>
-         </geometry>
-	   </collision>
    </link>
    <joint name="gripper_camera_visu_joint" type="fixed" >
@@ -183,9 +163,4 @@
          </material>
       </visual>
-      <collision>
-         <geometry>
-            <box size="0.00 0.00 0.0"/>
-         </geometry>
-	   </collision>
    </link>
   </xacro:macro>

File: franka_description/robots/hand.xacro (robot description, xacro)
@@ -118,9 +118,4 @@
 	      <material name="silver" />
       </visual>
-      <collision>
-         <geometry>
-            <box size="0.00 0.00 0.0"/>
-         </geometry>
-	   </collision>
    </link>
    <joint name="realsense_camera_joint" type="fixed" >
@@ -136,14 +131,9 @@
 	      <material name="silver" />
       </visual>
-      <collision>
-         <geometry>
-            <box size="0.00 0.00 0.0"/>
-         </geometry>
-	   </collision>
    </link>
-      <joint name="gripper_realsense_joint" type="fixed" >
-      <parent link="${ns}_hand" />
-      <child link="camera_link" />
-     <origin xyz=" -0.039278 -0.012625  0.076519" rpy= "${180*pi/180} ${-90*pi/180} 0.0" />
+    <joint name="gripper_realsense_joint" type="fixed" >
+    <parent link="${ns}_hand" />
+    <child link="camera_link" />
+    <origin xyz=" -0.039278 -0.012625  0.076519" rpy= "${180*pi/180} ${-90*pi/180} 0.0" />
      <!-- "${-1.049392*pi/180} ${-4.432421*pi/180} ${91.376356*pi/180}" -->
      <!--"0.033641884557 -0.013806793567 1.57762792946"  -->
@@ -156,9 +146,4 @@
 	      <material name="silver" />
       </visual>
-      <collision>
-         <geometry>
-            <box size="0.00 0.00 0.0"/>
-         </geometry>
-	   </collision>
    </link>
    <joint name="gripper_camera_visu_joint" type="fixed" >
@@ -176,9 +161,4 @@
          </material>
       </visual>
-      <collision>
-         <geometry>
-            <box size="0.00 0.00 0.0"/>
-         </geometry>
-	   </collision>
    </link>
   </xacro:macro>
