Commit message: collision disable

File: franka_description/robots/end_effector/hand.xacro (robot description, xacro)
@@ -95,12 +95,6 @@
           <box size="0.0 0.00 0.0"/>
         </geometry>
-	<material name="silver" />
+	      <material name="silver" />
       </visual>
-      <collision>
-        <geometry>
-          <box size="0.00 0.00 0.0"/>
-        </geometry>
-	<material name="black"/>
-     </collision>
     </link>
   </xacro:macro>

File: franka_description/robots/hand.xacro (robot description, xacro)
@@ -87,5 +87,5 @@
       <parent link="${ns}_hand" />
       <child link="${ns}_object_link" />
-      <origin xyz="0 0 0.170" rpy="0 0 0"/>
+      <origin xyz="0 0 0.1034" rpy="0 0 0"/>
       <!-- Base delle dita 0.0584-->
    </joint>

File: panda_moveit_config/config/hand.xacro (robot description, xacro)
@@ -20,4 +20,5 @@
     <disable_collisions link1="panda_hand" link2="panda_rightfinger" reason="Adjacent" />
     <disable_collisions link1="panda_leftfinger" link2="panda_rightfinger" reason="Default" />
+    <disable_collisions link1="panda_object_link" link2="panda_hand" reason="Default" />
     <disable_collisions link1="panda_object_link" link2="panda_tactile_link" reason="Default" />
     <disable_collisions link1="panda_hand" link2="camera_link" reason="Default" />

File: panda_moveit_config/config/panda_arm_hand.srdf.xacro (robot description, xacro)
@@ -30,4 +30,5 @@
   <!--DISABLE COLLISIONS: By default it is assumed that any link of the robot could potentially come into collision with any other link in the robot. This tag disables collision checking between a specified pair of links. -->
   <disable_collisions link1="panda_hand" link2="panda_link4" reason="Never" />
+  <disable_collisions link1="panda_hand" link2="panda_link5" reason="Never" />
   <disable_collisions link1="panda_hand" link2="panda_link6" reason="Never" />
   <disable_collisions link1="panda_hand" link2="panda_link7" reason="Default" />
